Commit message: Using three types of environments to test the effectiveness of our planning and execution

File: urdfenvs/assets/home/basket.urdf (robot description, URDF)
Before this commit: robot banana, 1 links, 0 joints
Links:
- removed link banana_base_link
- added link basket_base_link, mass 1.0; collision mesh filename=package://meshes/basket.dae scale=1 1 1; visual mesh filename=package://meshes/basket.dae scale=1 1 1
