Commit message: Adjusted table dimensions to include objects as well as albert base within the table

File: urdfenvs/assets/maze/maze.urdf (robot description, URDF)
Before this commit: robot random_environment, 20 links, 19 joints
Links:
- added link table_2_3, mass .0; collision box size=1.5 1 0.05; visual mesh filename=table.obj scale=0.1 0.1 0.75
Joints:
- added joint joint_table_2_3: type fixed, parent world, child table_2_3, origin xyz=2.3 0.5833333333333339 0.0 rpy=0 0 0

File: urdfenvs/assets/supermarket/supermarket_instance_1.urdf (robot description, URDF)
Before this commit: robot supermarket, 17 links, 16 joints
Links:
- link table_2_3: geometry collision box size=1.5 1 0.05; visual mesh filename=table.obj scale=0.1 0.1 0.75

Commit message: Removed table urdf as it was separately loaded as an obstacle

File: urdfenvs/assets/maze/maze.urdf (robot description, URDF)
Before this commit: robot random_environment, 21 links, 20 joints
Links:
- removed link table_2_3
Joints:
- removed joint joint_table_2_3

File: urdfenvs/assets/supermarket/supermarket_instance_1.urdf (robot description, URDF)
Before this commit: robot supermarket, 17 links, 16 joints
Links:
- removed link table_2_3
Joints:
- removed joint joint_table_2_3
